Commit message: support rgb depth camera in lerobot sim

File: ROS2/lerobot_ws/src/lerobot_description/urdf/so101_base.xacro (robot description, xacro)
@@ -447,3 +447,39 @@
 		</actuator>
 	</transmission>
+	<!-- Depth Camera Link -->
+	<link name="camera_link">
+		<inertial>
+			<origin xyz="0 0 0" rpy="0 0 0"/>
+			<mass value="0.1"/>
+			<inertia ixx="0.0001" ixy="0" ixz="0" iyy="0.0001" iyz="0" izz="0.0001"/>
+		</inertial>
+		<visual>
+			<origin xyz="0 0 0" rpy="0 0 0"/>
+			<geometry>
+				<box size="0.05 0.05 0.03"/>
+			</geometry>
+			<material name="camera_material">
+				<color rgba="0.2 0.2 0.2 1.0"/>
+			</material>
+		</visual>
+		<collision>
+			<origin xyz="0 0 0" rpy="0 0 0"/>
+			<geometry>
+				<box size="0.05 0.05 0.03"/>
+			</geometry>
+		</collision>
+	</link>
+	<!-- Camera Joint - Mount camera above the workspace -->
+	<joint name="camera_joint" type="fixed">
+		<parent link="world"/>
+		<child link="camera_link"/>
+		<origin xyz="0.0 0.0 1.5" rpy="0 1.57 0"/>
+	</joint>
+	<!-- Optical Frame (for proper camera orientation) -->
+	<link name="camera_optical_link"/>
+	<joint name="camera_optical_joint" type="fixed">
+		<parent link="camera_link"/>
+		<child link="camera_optical_link"/>
+		<origin xyz="0 0 0" rpy="-1.5708 0 -1.5708"/>
+	</joint>
 </robot>

File: ROS2/lerobot_ws/src/lerobot_description/urdf/so101_gazebo.xacro (robot description, xacro)
@@ -7,3 +7,51 @@
         </plugin>
     </gazebo>
+    <!-- Sensors System Plugin - REQUIRED for Ignition Gazebo -->
+    <gazebo>
+        <plugin filename="libignition-gazebo-sensors-system.so" name="ignition::gazebo::systems::Sensors">
+            <render_engine>ogre2</render_engine>
+        </plugin>
+    </gazebo>
+    <!-- RGB Camera -->
+    <gazebo reference="camera_link">
+        <sensor name="camera" type="camera">
+            <always_on>true</always_on>
+            <update_rate>30</update_rate>
+            <visualize>true</visualize>
+            <frame_id>camera_optical_link</frame_id>
+            <camera>
+                <horizontal_fov>1.047198</horizontal_fov>
+                <image>
+                    <width>640</width>
+                    <height>480</height>
+                    <format>R8G8B8</format>
+                </image>
+                <clip>
+                    <near>0.1</near>
+                    <far>5.0</far>
+                </clip>
+            </camera>
+        </sensor>
+    </gazebo>
+    <!-- Depth Camera -->
+    <gazebo reference="camera_link">
+        <sensor name="depth_camera" type="depth_camera">
+            <always_on>true</always_on>
+            <update_rate>10</update_rate>
+            <visualize>true</visualize>
+            <frame_id>camera_optical_link</frame_id>
+            <camera>
+                <horizontal_fov>1.047198</horizontal_fov>
+                <image>
+                    <width>640</width>
+                    <height>480</height>
+                    <format>R_FLOAT32</format>
+                </image>
+                <clip>
+                    <near>0.1</near>
+                    <far>2</far>
+                </clip>
+            </camera>
+        </sensor>
+    </gazebo>
 </robot>
